File: electronic/garland_controller.kicad_pcb (KiCad board)
At the start: 2 copper layers, 40 x 25 mm, 31 parts, among them J1 USB_C_Receptacle_USB2.0_16P, J2 Conn_01x03_Socket, J3 Conn_01x05_Pin, J4 Conn_01x03_Pin, U1 USBLC6-2SC6, U2 STM32F103C8Tx, U3 AMS1117-3.3, Y1 8MHz

Commit message: Tune fuses
Parts:
- added H1: MountingHole, MountingHole:MountingHole_2.1mm, F.Cu at (113.0, 62.0)
- added H2: MountingHole, MountingHole:MountingHole_2.1mm, F.Cu at (104.0, 77.0)
- added H3: MountingHole, MountingHole:MountingHole_2.1mm, F.Cu at (137.0, 64.0)
- D2: value ESD5Zxx -> ESD5Z3V3
- F1: value Polyfuse -> 3A; footprint Fuse:Fuse_1206_3216Metric_Pad1.42x1.75mm_HandSolder -> Fuse:Fuse_1210_3225Metric_Pad1.42x2.65mm_HandSolder
- F2: value Polyfuse -> 60mA; footprint Fuse:Fuse_1206_3216Metric_Pad1.42x1.75mm_HandSolder -> Fuse:Fuse_0805_2012Metric_Pad1.15x1.40mm_HandSolder
- moved G1 39.8 mm to (83.0, 68.0)
- moved U1 11.2 mm to (110.9, 69.0)
- moved R5 8.25 mm to (109.0, 61.0)
- moved R3 7.00 mm to (111.0, 66.0), turned to 180 degrees
- moved R4 6.46 mm to (106.0, 60.9)
- moved C2 4.47 mm to (122.0, 65.0)
- moved U2 4.00 mm to (129.0, 64.0)
- moved F2 3.61 mm to (109.0, 74.0)
- moved R6 2.28 mm to (123.0, 60.0)
- moved C3 2.00 mm to (127.1, 57.0)
- moved D2 1.41 mm to (119.3, 61.0)
- moved J4 1.00 mm to (110.5, 57.0)
- moved J2 1.00 mm to (115.5, 57.0)
- moved J1 0.50 mm to (103.0, 67.5)
- turned C9 to 180 degrees

Commit message: Layout rev. 0.1
Parts:
- added TP1: TestPoint, Connector_PinHeader_2.54mm:PinHeader_1x01_P2.54mm_Vertical, F.Cu at (130.0, 56.5)
- G1: moved to B.Cu
- moved G1 41.9 mm to (124.8, 64.2), turned to 180 degrees
- moved R4 16.7 mm to (107.5, 77.5), turned to -90 degrees
- moved R3 11.7 mm to (122.5, 64.0), turned to 90 degrees
- moved C8 6.02 mm to (136.0, 78.5), turned to 180 degrees
- moved C10 5.52 mm to (109.5, 74.5)
- moved C7 5.27 mm to (123.5, 73.5), turned to 180 degrees
- moved F2 4.27 mm to (110.5, 70.0), turned to 0 degrees
- moved C11 4.03 mm to (121.5, 70.0), turned to -90 degrees
- moved C9 4.03 mm to (130.0, 78.5), turned to 0 degrees
- moved C5 2.85 mm to (134.5, 68.5)
- moved U3 2.55 mm to (116.5, 70.5)
- moved R6 2.50 mm to (120.5, 60.0)
- moved U1 2.45 mm to (110.9, 66.5)
- moved D2 2.33 mm to (117.2, 60.0), turned to 180 degrees
- moved R5 2.15 mm to (106.9, 60.5), turned to 180 degrees
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Connections:
- net /USB_DM renamed /USB_D+
- net /USB_DP renamed /USB_D-
- U2 pad 28: unconnected-(U2-PB15-Pad28) -> /DEBUG_LED
- U2 pad 31: /USB_ON -> unconnected-(U2-PA10-Pad31)
- U2 pad 43: /DEBUG_LED -> /USB_ON
Routing:
- net +3V3: track 0.00 -> 94.1 mm, vias 0 -> 8
- net GND: track 0.00 -> 50.4 mm, vias 0 -> 29
- net +5V: track 0.00 -> 36.9 mm
- net Net-(J3-Pin_2): track 0.00 -> 27.8 mm, vias 0 -> 2
- net Net-(J3-Pin_3): track 0.00 -> 24.7 mm, vias 0 -> 2
- net /USB_D-: track 0.00 -> 21.5 mm
- net /USB_D+: track 0.00 -> 20.6 mm
- net /NRST: track 0.00 -> 16.4 mm, vias 0 -> 2
- net Net-(J2-Pin_1): track 0.00 -> 15.0 mm
- net Net-(U3-VI): track 0.00 -> 13.4 mm
- net Net-(U2-PD0): track 0.00 -> 12.5 mm
- net Net-(J1-CC2): track 0.00 -> 10.2 mm, vias 0 -> 2
- net Net-(C8-Pad1): track 0.00 -> 9.17 mm
- net Net-(J1-CC1): track 0.00 -> 7.32 mm
- net /DEBUG_LED: track 0.00 -> 6.27 mm
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- added copper zone on B.Cu, net GND
- added copper zone on F.Cu, net GND
Other:
- board text added: "Garland controller rev. 0.1"
